File: DUMDUMDrUmMachine/7seg&Buttons.sch (EAGLE design)
At the start: 6 parts

Commit message: 7sge&buttons schematics finnished
Parts:
- added R1, R10, R11, R12, R13, R14, R15, R16, R17, R18, R2, R3, R4, R5, R6, R7, R8: 20K, resistor:R-EU_0204/7
- added R9: 100, resistor:R-EU_0204/7
- added S1, S10, S11, S12, S13, S14, S15, S16, S2, S3, S4, S5, S6, S7, S8, S9: (no value), switch-omron:40-XX
- added V4, V5: 74165N, 74ttl-din:74165N
Connections:
- net CLOCK_IN_PIN renamed CLOCK_PIN_164
- removed net 5V: DIS1.CA, DIS1.CA@1, DIS2.CA, DIS2.CA@1, DIS3.CA, DIS3.CA@1, V11.!CLR, V21.!CLR, V31.!CLR
- new net +5V: DIS3.CA, DIS3.CA@1, R1.2, R10.2, R11.2, R12.2, R13.2, R14.2, R15.2, R16.2, R17.2, R18.2, R2.2, R3.2, R4.2, R5.2, R6.2, R7.2, R8.2, R9.2, V1/+UB.+UB, V11.!CLR, V2/+UB.+UB, V21.!CLR, V3/+UB.+UB, V31.!CLR, V4/+UB.+UB
- new net CLOCK_PIN_165: V41.CLK, V41.CLK_INH, V51.CLK, V51.CLK_INH
- new net GND: S1.P, S1.P1, S10.P, S10.P1, S11.P, S11.P1, S12.P, S12.P1, S13.P, S13.P1, S14.P, S14.P1, S15.P, S15.P1, S16.P, S16.P1, S2.P, S2.P1, S3.P, S3.P1, S4.P, S4.P1, S5.P, S5.P1, S6.P, S6.P1, S7.P, S7.P1, S8.P, S8.P1, S9.P, S9.P1, V1/-UB.-UB, V2/-UB.-UB, V3/-UB.-UB, V4/-UB.-UB
- new net N$16: DIS1.CA, DIS1.CA@1, R9.1
- new net N$23: DIS2.CA, DIS2.CA@1, R10.1
- new net N$24: R18.1, S16.S, S16.S1, V51.H
- new net N$25: R17.1, S15.S, S15.S1, V51.G
- new net N$26: R16.1, S14.S, S14.S1, V51.F
- new net N$27: R15.1, S13.S, S13.S1, V51.E
- new net N$28: R14.1, S12.S, S12.S1, V51.D
- new net N$29: R13.1, S11.S, S11.S1, V51.C
- new net N$30: R8.1, S8.S, S8.S1, V41.H
- new net N$31: R7.1, S7.S, S7.S1, V41.G
- new net N$32: R6.1, S6.S, S6.S1, V41.F
- new net N$33: R5.1, S5.S, S5.S1, V41.E
- new net N$34: R4.1, S4.S, S4.S1, V41.D
- new net N$35: R3.1, S3.S, S3.S1, V41.C
- new net N$36: R2.1, S2.S, S2.S1, V41.B
- new net N$37: R1.1, S1.S, S1.S1, V41.A
- new net N$38: R12.1, S10.S, S10.S1, V51.B
- new net N$39: R11.1, S9.S, S9.S1, V51.A
- new net N$40: V41.QH, V51.SER
- new net PL_PIN_165: V41.SH/!LD, V51.SH/!LD
- new net SERIAL_INPUT_165: V51.QH
Other:
- note added: "This diasy-chain is not tested to acually work with the code, yet"
