File: Eagle-files, gerbers & chaos/ACC+PWM-CV.brd (EAGLE design)
At the start: 100 x 80 mm, 58 parts, among them IC1 TL072P, IC4 7815T, IC6 4584N, IC7 7805T, X1 5 VDC, X2 15 VAC, X3 NOISE_OUT

Commit message: Cleaned up, added PDF of schematics
Parts:
- removed C15: 22n, rcl:C075-042X103
- removed C16, C17, C20: 19n, rcl:C075-042X103
- removed C18, C19: 10n, rcl:C075-042X103
- removed C21, C22: 1u, rcl:E5-6
- removed IC6: 4584N, 45xx:DIL14
- removed IC7: 7805T, linear:TO220H
- removed JMP1, JMP2, JMP4: 0, rcl:0207/10
- removed JMP3: 0, rcl:0207/12
- removed PWR_OUT1, PWR_OUT2, PWR_OUT3, PWR_OUT4: +15V, GND, -15V, con-ptr500:AK300/3
- removed R18, R19: 120k, rcl:0207/5V
- added C6: 100n, rcl:C075-042X103
- added C7, C8: 1u, rcl:C075-042X103
- added IC2: TL072P, linear:DIL08
- added IC3: TL071P, linear:DIL08
- added R11, R12: 1K, rcl:0207/10
- added X4: PWM, con-ptr500:AK300/2
- added X5: CV, con-ptr500:AK300/2
- C1: value 1n -> 100n
- C2, C3: value 3.3n -> 100n
- C4, C5: value 0.1u -> 100n
- R1: value 300k -> 500K?; device rcl:0207/5V -> rcl:PT-10
- R10: value 82k -> 1K; device rcl:0207/5V -> rcl:0207/10
- R13: device rcl:0207/5V -> rcl:0207/10
- R14: value 120k -> 1.2k; device rcl:0207/5V -> rcl:0207/10
- R15: value 560k -> valfri; device rcl:0207/5V -> rcl:0207/10
- R16: value 120k -> valfri; device rcl:0207/5V -> rcl:0207/10
- R17: value 560 -> 1.2k; device rcl:0207/5V -> rcl:0207/10
- R2: value 120k -> 20K; device rcl:0207/5V -> rcl:0207/10
- R3: value 270k -> 10K; device rcl:0207/5V -> rcl:0207/10
- R4: value 120k -> 1K; device rcl:0207/5V -> rcl:0207/10
- R5: value 220k -> 1K; device rcl:0207/5V -> rcl:0207/10
- R6: value 120k -> 15K; device rcl:0207/5V -> rcl:0207/10
- R7: value 680k -> 1K; device rcl:0207/5V -> rcl:0207/10
- R8: value 22k -> 1K; device rcl:0207/5V -> rcl:0207/10
- R9: value 580 -> 1K; device rcl:0207/5V -> rcl:0207/10
- X1: value 5 VDC -> ACC_IN
- X3: value NOISE_OUT -> ACC_OUT
- moved R6 75.0 mm to (73.7, 38.1), turned to 270 degrees
- moved R4 62.7 mm to (63.5, 38.1), turned to 270 degrees
- moved R5 61.4 mm to (66.0, 38.1), turned to 270 degrees
- moved R1 60.7 mm to (71.1, 6.35), turned to 90 degrees
- moved R3 59.7 mm to (72.4, 14.0)
- moved R2 59.3 mm to (63.5, 12.7), turned to 270 degrees
- moved R8 55.0 mm to (58.4, 74.9), turned to 180 degrees
- moved R10 52.8 mm to (67.3, 69.8), turned to 90 degrees
- moved IC5 47.2 mm to (14.0, 45.7), turned to 90 degrees
- moved C5 45.9 mm to (53.3, 52.1), turned to 180 degrees
- moved R7 45.9 mm to (69.8, 38.1), turned to 270 degrees
- moved PWR_OUT 45.8 mm to (31.8, 6.35)
- moved R9 44.5 mm to (58.4, 72.4), turned to 180 degrees
- moved C11 44.5 mm to (33.0, 17.8), turned to 0 degrees
- moved X1 42.2 mm to (54.6, 8.89), turned to 0 degrees
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Connections:
- removed net +5V: C22.+, IC7.3, JMP2.2, X1.1
- removed net N$15: C18.1, IC6.9, R7.2
- removed net N$16: C17.1, IC6.5, R5.2
- removed net N$17: C16.1, IC6.3, R3.2
- removed net N$18: C15.1, IC6.1, R1.2
- removed net N$21: IC1.6, IC1.7
- removed net N$25: IC6.14, JMP2.1
- removed net N$27: IC1.4, JMP4.1
- removed net N$28: C4.1, IC1.8, JMP3.1
- net +15V: now also C1.2, C3.2, C5.2, IC1.8, IC2.8, IC3.7, R14.2; no longer C21.+, IC7.1, JMP3.2, PWR_OUT1.1, PWR_OUT2.1, PWR_OUT3.1, PWR_OUT4.1
- net -15V: now also C2.1, C4.1, C6.1, IC1.4, IC2.4, IC3.4, R17.1, R6.1; no longer C5.2, JMP4.2, PWR_OUT1.3, PWR_OUT2.3, PWR_OUT3.3, PWR_OUT4.3
- net GND: now also C1.1, C2.2, C3.1, C6.2, C8.1, IC2.5, R1.1, R10.1, R12.1, R15.1, R16.2, R3.1, X4.2, X5.2; no longer C15.2, C16.2, C17.2, C18.2, C19.2, C20.2, C21.-, C22.-, IC1.3, IC1.5, IC6.7, IC7.2, PWR_OUT1.2, PWR_OUT2.2, PWR_OUT3.2, PWR_OUT4.2, R19.2, R9.2
- net N$1: now also IC2.1, IC2.2, R1.2; no longer C1.2, R14.1, R16.1, R18.1, R19.1, R2.1, R4.1, R6.1
- net N$10: now also R8.2, X4.1; no longer C10.-, D2.A, JMP1.2
- net N$11: now also R10.2, R8.1, R9.2; no longer C1.1, R8.2
- net N$12: now also C7.2, C8.2, IC3.3, R9.1; no longer C2.2, IC1.2, R10.1, R8.1
- net N$13: now also C7.1, IC3.6, R11.1, X5.1; no longer C3.1, IC1.1, R10.2, X3.1
- net N$14: now also IC3.2, R11.2, R12.2; no longer C2.1, C3.2, R9.1
- net N$2: now also IC1.3, R1.3; no longer IC6.12, R17.1, R18.2
- net N$23: now also C10.-, D2.A; no longer JMP1.1
- net N$24: now also R14.1, R15.2
- net N$26: now also R16.1, R17.2
- net N$3: now also IC1.1, IC1.5, R2.2; no longer IC6.10, R15.1, R16.2
- net N$4: now also IC1.2, R2.1, R3.2; no longer IC6.8, R14.2, R7.1
- net N$5: now also IC2.7, R7.2; no longer IC6.6, R6.2
- net N$6: now also IC2.6, R6.2, R7.1; no longer IC6.4, R3.1, R4.2
- net N$7: now also IC1.6, R4.1, R5.2; no longer IC6.2, R1.1, R2.2
- net N$8: now also IC1.7, R4.2, X3.1; no longer C20.1, IC6.13, R17.2
- net N$9: now also IC2.3, X1.1; no longer C19.1, IC6.11, R15.2
Routing:
- net GND: track 539.0 -> 390.7 mm, vias 0 -> 7
- net N$1: track 87.0 -> 14.5 mm
- net +5V: track 53.5 -> 0.00 mm
- net N$28: track 49.6 -> 0.00 mm
- net N$8: track 15.3 -> 50.1 mm
- net N$22: track 35.2 -> 62.9 mm
- net N$24: track 40.6 -> 13.8 mm
- net N$9: track 14.3 -> 38.8 mm, vias 0 -> 1
- net N$27: track 19.9 -> 0.00 mm
- net N$23: track 16.1 -> 35.4 mm
- net N$14: track 11.7 -> 30.4 mm
- net N$25: track 15.4 -> 0.00 mm
- net N$18: track 14.3 -> 0.00 mm, vias 0 -> 1
- net N$16: track 12.8 -> 0.00 mm, vias 0 -> 1
- net N$15: track 12.5 -> 0.00 mm, vias 0 -> 1
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- removed copper zone on layer 16, net GND
Other:
- board text removed: "DUMDUM Double sun POWER"
